Commit message: .

File: urdf/farm-ng_test.xacro (robot description, xacro)
@@ -1,9 +1,10 @@
 <?xml version="1.0"?>
 <robot xmlns:xacro="http://www.ros.org/wiki/xacro" name="amiga">
+ <!--xacro:include filename="$(find amiga_cmu_description)/urdf/farm-ng.gazebo"/-->
 <link name="base_footprint"/>
 <link name="base_link">
     <inertial>
         <origin xyz="0.0 0.0 0.22" rpy="0.0 0.0 0.0"/>
-        <mass value="1.0"/>
+        <mass value="10.0"/>
         <inertia ixx="0.4" ixy="0.0" ixz="0.0"
                  iyy="0.4" iyz="0.0"
@@ -40,5 +41,5 @@
         <inertial>
             <origin xyz="0.0 0.0 0.0" rpy="0.0 0.0 0.0"/>
-            <mass value="0.5"/>
+            <mass value="1"/>
             <inertia ixx="0.0" ixy="0.0" ixz="0.0" iyy="0.0" iyz="0.0" izz="0.0"/>
         </inertial>
@@ -75,5 +76,5 @@
         <inertial>
             <origin xyz="0.0 0.0 0.0" rpy="0.0 0.0 0.0"/>
-            <mass value="0.5"/>
+            <mass value="1"/>
             <inertia ixx="0.1" ixy="0.0" ixz="0.0" iyy="0.1" iyz="0.0" izz="0.1"/>
         </inertial>
@@ -145,4 +146,28 @@
     geometry_mesh_origin_xyz="$(arg geometry_mesh_origin_xyz)" geometry_mesh_origin_rpy="$(arg geometry_mesh_origin_rpy)"
     geometry_mesh_tcp_xyz="$(arg geometry_mesh_tcp_xyz)" geometry_mesh_tcp_rpy="$(arg geometry_mesh_tcp_rpy)" />
-    <xacro:include filename="$(find amiga_cmu_description)/urdf/farm-ng.gazebo"/>
+<gazebo>
+    <plugin name="skid_steer_drive_controller" filename="libgazebo_ros_skid_steer_drive.so">
+      <updateRate>10.0</updateRate>
+      <robotNamespace>/</robotNamespace>
+      <leftFrontJoint>tire_front_left_joint</leftFrontJoint>
+      <rightFrontJoint>tire_front_right_joint</rightFrontJoint>
+      <leftRearJoint>tire_rear_left_joint</leftRearJoint>
+      <rightRearJoint>tire_rear_right_joint</rightRearJoint>
+      <wheelSeparation>1.2192</wheelSeparation>
+      <wheelDiameter>0.22</wheelDiameter>
+      <robotBaseFrame>base_link</robotBaseFrame>
+      <torque>10</torque>
+      <topicName>cmd_vel</topicName>
+      <odometryTopic>odom</odometryTopic>
+      <odometryFrame>odom</odometryFrame>
+      <commandTopic>cmd_vel</commandTopic>
+      <topic_name_twist>cmd_vel</topic_name_twist>
+      <topic_name_odometry>odom</topic_name_odometry>
+      <topic_name_joint>joint</topic_name_joint>
+      <broadcastTF>true</broadcastTF>
+      <covariance_x>0.0001</covariance_x>
+      <covariance_y>0.0001</covariance_y>
+      <covariance_yaw>0.01</covariance_yaw>
+    </plugin>
+  </gazebo>
 </robot>
