Commit message: .

File: urdf/farm-ng.urdf.xacro (robot description, xacro)
@@ -35,4 +35,73 @@
     <axis xyz="0.0 0.0 0.0"/>
 </joint>
+<!-- All crossbeams links and joints -->
+<xacro:macro name="Lcrossbeam" params="name x y">
+    <link name="Lcrossbeam_${name}_link">
+        <inertial>
+            <origin xyz="0.0 0.0 0.0" rpy="0.0 0.0 0.0"/>
+            <mass value="0.5"/>
+            <inertia ixx="0.0" ixy="0.0" ixz="0.0" iyy="0.0" iyz="0.0" izz="0.0"/>
+        </inertial>
+        <visual name="">
+            <origin xyz="0.0 0.0 0.0" rpy="0.0 0.0 0.0"/>
+            <geometry>
+                <mesh filename="package://amiga_cmu_description/meshes/LCrossbeam/LCrossbeam.obj" scale="1.0 1.3 1.0"/>
+            </geometry>
+            <material name="black">
+                <color rgba=".0 .0 0.0 1.0"/>
+            </material>
+        </visual>
+        <collision>
+            <origin xyz="0.0 0.0 0.0" rpy="0.0 0.0 0.0"/>
+            <geometry>
+                <mesh filename="package://amiga_cmu_description/meshes/LCrossbeam/LCrossbeam.obj" scale="1.0 1.3 1.0"/>
+            </geometry>
+        </collision>
+    </link>
+    <joint name="Lcrossbeam_${name}_joint" type="fixed">
+        <origin xyz="${x} ${y} .66" rpy="0 0.0 0.0"/>
+        <parent link="base_link"/>
+        <child link="Lcrossbeam_${name}_link"/>
+        <axis xyz="0.0 0.0 0.0"/>
+    </joint>
+</xacro:macro>
+<xacro:Lcrossbeam name="front1"  x="0.525" y =" 0.0"/>
+<xacro:Lcrossbeam name="front2"  x="0.6942" y =" 0.0"/>
+<xacro:Lcrossbeam name="back1"  x="-0.525" y =" 0.0"/>
+<xacro:Lcrossbeam name="back2"  x="-0.6942" y =" 0.0"/>
+<xacro:macro name="Wcrossbeam" params="name x y">
+    <link name="Wcrossbeam_${name}_link">
+        <inertial>
+            <origin xyz="0.0 0.0 0.0" rpy="0.0 0.0 1.571"/>
+            <mass value="0.5"/>
+            <inertia ixx="0.0" ixy="0.0" ixz="0.0" iyy="0.0" iyz="0.0" izz="0.0"/>
+        </inertial>
+        <visual name="">
+            <origin xyz="0.0 0.0 0.0" rpy="0.0 0.0 1.571"/>
+            <geometry>
+                <mesh filename="package://amiga_cmu_description/meshes/WCrossbeam/WCrossbeam.obj" scale="1.0 1.2 1.0"/>
+            </geometry>
+            <material name="black">
+                <color rgba=".0 .0 0.0 1.0"/>
+            </material>
+        </visual>
+        <collision>
+            <origin xyz="0.0 0.0 0.0" rpy="0.0 0.0 1.571"/>
+            <geometry>
+                <mesh filename="package://amiga_cmu_description/meshes/WCrossbeam/WCrossbeam.obj" scale="1.0 1.2 1.0"/>
+            </geometry>
+        </collision>
+    </link>
+    <joint name="Wcrossbeam_${name}_joint" type="fixed">
+        <origin xyz="${x} ${y} .36" rpy="0 0.0 0.0"/>
+        <parent link="base_link"/>
+        <child link="Wcrossbeam_${name}_link"/>
+        <axis xyz="0.0 0.0 0.0"/>
+    </joint>
+</xacro:macro>
+<xacro:Wcrossbeam name="left1"  x="0.0" y =" 0.70"/>
+<xacro:Wcrossbeam name="left2"  x="0.0" y =" 0.824"/>
+<xacro:Wcrossbeam name="right1"  x="0.0" y =" -0.70"/>
+<xacro:Wcrossbeam name="right2"  x="0.0" y =" -0.824"/>
 <!-- All Wheel links and joints -->
 <xacro:macro name="wheel" params="name x y">
@@ -111,5 +180,5 @@
   <xacro:arg name="velocity_control" default="false"/>
   <xacro:arg name="attach_to" default="base_link"/>
-  <xacro:arg name="xyz" default="0 -0.762 0.65"/>
+  <xacro:arg name="xyz" default="0 -0.762 0.385"/>
   <xacro:arg name="rpy" default="0 0 -1.5"/>
   <xacro:arg name="add_other_geometry" default="false"/>

File: urdf/farm-ng_test.xacro (robot description, xacro)
@@ -36,4 +36,73 @@
     <axis xyz="0.0 0.0 0.0"/>
 </joint>
+<!-- All crossbeams links and joints -->
+<xacro:macro name="Lcrossbeam" params="name x y">
+    <link name="Lcrossbeam_${name}_link">
+        <inertial>
+            <origin xyz="0.0 0.0 0.0" rpy="0.0 0.0 0.0"/>
+            <mass value="0.5"/>
+            <inertia ixx="0.0" ixy="0.0" ixz="0.0" iyy="0.0" iyz="0.0" izz="0.0"/>
+        </inertial>
+        <visual name="">
+            <origin xyz="0.0 0.0 0.0" rpy="0.0 0.0 0.0"/>
+            <geometry>
+                <mesh filename="package://amiga_cmu_description/meshes/LCrossbeam/LCrossbeam.obj" scale="1.0 1.3 1.0"/>
+            </geometry>
+            <material name="black">
+                <color rgba=".0 .0 0.0 1.0"/>
+            </material>
+        </visual>
+        <collision>
+            <origin xyz="0.0 0.0 0.0" rpy="0.0 0.0 0.0"/>
+            <geometry>
+                <mesh filename="package://amiga_cmu_description/meshes/LCrossbeam/LCrossbeam.obj" scale="1.0 1.3 1.0"/>
+            </geometry>
+        </collision>
+    </link>
+    <joint name="Lcrossbeam_${name}_joint" type="fixed">
+        <origin xyz="${x} ${y} .66" rpy="0 0.0 0.0"/>
+        <parent link="base_link"/>
+        <child link="Lcrossbeam_${name}_link"/>
+        <axis xyz="0.0 0.0 0.0"/>
+    </joint>
+</xacro:macro>
+<xacro:Lcrossbeam name="front1"  x="0.525" y =" 0.0"/>
+<xacro:Lcrossbeam name="front2"  x="0.6942" y =" 0.0"/>
+<xacro:Lcrossbeam name="back1"  x="-0.525" y =" 0.0"/>
+<xacro:Lcrossbeam name="back2"  x="-0.6942" y =" 0.0"/>
+<xacro:macro name="Wcrossbeam" params="name x y">
+    <link name="Wcrossbeam_${name}_link">
+        <inertial>
+            <origin xyz="0.0 0.0 0.0" rpy="0.0 0.0 1.571"/>
+            <mass value="0.5"/>
+            <inertia ixx="0.0" ixy="0.0" ixz="0.0" iyy="0.0" iyz="0.0" izz="0.0"/>
+        </inertial>
+        <visual name="">
+            <origin xyz="0.0 0.0 0.0" rpy="0.0 0.0 1.571"/>
+            <geometry>
+                <mesh filename="package://amiga_cmu_description/meshes/WCrossbeam/WCrossbeam.obj" scale="1.0 1.2 1.0"/>
+            </geometry>
+            <material name="black">
+                <color rgba=".0 .0 0.0 1.0"/>
+            </material>
+        </visual>
+        <collision>
+            <origin xyz="0.0 0.0 0.0" rpy="0.0 0.0 1.571"/>
+            <geometry>
+                <mesh filename="package://amiga_cmu_description/meshes/WCrossbeam/WCrossbeam.obj" scale="1.0 1.2 1.0"/>
+            </geometry>
+        </collision>
+    </link>
+    <joint name="Wcrossbeam_${name}_joint" type="fixed">
+        <origin xyz="${x} ${y} .36" rpy="0 0.0 0.0"/>
+        <parent link="base_link"/>
+        <child link="Wcrossbeam_${name}_link"/>
+        <axis xyz="0.0 0.0 0.0"/>
+    </joint>
+</xacro:macro>
+<xacro:Wcrossbeam name="left1"  x="0.0" y =" 0.70"/>
+<xacro:Wcrossbeam name="left2"  x="0.0" y =" 0.824"/>
+<xacro:Wcrossbeam name="right1"  x="0.0" y =" -0.70"/>
+<xacro:Wcrossbeam name="right2"  x="0.0" y =" -0.824"/>
 <!-- All Wheel links and joints -->
 <xacro:macro name="wheel" params="name x y">
@@ -114,5 +183,5 @@
   <xacro:arg name="velocity_control" default="false"/>
   <xacro:arg name="attach_to" default="base_link"/>
-  <xacro:arg name="xyz" default="0 -0.762 0.65"/>
+  <xacro:arg name="xyz" default="0 -0.762 0.385"/>
   <xacro:arg name="rpy" default="0 0 -1.5"/>
   <xacro:arg name="add_other_geometry" default="false"/>

Commit message: .

File: urdf/farm-ng.urdf.xacro (robot description, xacro)
@@ -35,94 +35,25 @@
     <axis xyz="0.0 0.0 0.0"/>
 </joint>
-<!-- All crossbeams links and joints -->
-<xacro:macro name="Lcrossbeam" params="name x y">
-    <link name="Lcrossbeam_${name}_link">
-        <inertial>
-            <origin xyz="0.0 0.0 0.0" rpy="0.0 0.0 0.0"/>
-            <mass value="0.5"/>
-            <inertia ixx="0.0" ixy="0.0" ixz="0.0" iyy="0.0" iyz="0.0" izz="0.0"/>
-        </inertial>
-        <visual name="">
-            <origin xyz="0.0 0.0 0.0" rpy="0.0 0.0 0.0"/>
-            <geometry>
-                <mesh filename="package://amiga_cmu_description/meshes/LCrossbeam/LCrossbeam.obj" scale="1.0 1.3 1.0"/>
-            </geometry>
-            <material name="black">
-                <color rgba=".0 .0 0.0 1.0"/>
-            </material>
-        </visual>
-        <collision>
-            <origin xyz="0.0 0.0 0.0" rpy="0.0 0.0 0.0"/>
-            <geometry>
-                <mesh filename="package://amiga_cmu_description/meshes/LCrossbeam/LCrossbeam.obj" scale="1.0 1.3 1.0"/>
-            </geometry>
-        </collision>
-    </link>
-    <joint name="Lcrossbeam_${name}_joint" type="fixed">
-        <origin xyz="${x} ${y} .66" rpy="0 0.0 0.0"/>
-        <parent link="base_link"/>
-        <child link="Lcrossbeam_${name}_link"/>
-        <axis xyz="0.0 0.0 0.0"/>
-    </joint>
-</xacro:macro>
-<xacro:Lcrossbeam name="front1"  x="0.525" y =" 0.0"/>
-<xacro:Lcrossbeam name="front2"  x="0.6942" y =" 0.0"/>
-<xacro:Lcrossbeam name="back1"  x="-0.525" y =" 0.0"/>
-<xacro:Lcrossbeam name="back2"  x="-0.6942" y =" 0.0"/>
-<xacro:macro name="Wcrossbeam" params="name x y">
-    <link name="Wcrossbeam_${name}_link">
-        <inertial>
-            <origin xyz="0.0 0.0 0.0" rpy="0.0 0.0 1.571"/>
-            <mass value="0.5"/>
-            <inertia ixx="0.0" ixy="0.0" ixz="0.0" iyy="0.0" iyz="0.0" izz="0.0"/>
-        </inertial>
-        <visual name="">
-            <origin xyz="0.0 0.0 0.0" rpy="0.0 0.0 1.571"/>
-            <geometry>
-                <mesh filename="package://amiga_cmu_description/meshes/WCrossbeam/WCrossbeam.obj" scale="1.0 1.2 1.0"/>
-            </geometry>
-            <material name="black">
-                <color rgba=".0 .0 0.0 1.0"/>
-            </material>
-        </visual>
-        <collision>
-            <origin xyz="0.0 0.0 0.0" rpy="0.0 0.0 1.571"/>
-            <geometry>
-                <mesh filename="package://amiga_cmu_description/meshes/WCrossbeam/WCrossbeam.obj" scale="1.0 1.2 1.0"/>
-            </geometry>
-        </collision>
-    </link>
-    <joint name="Wcrossbeam_${name}_joint" type="fixed">
-        <origin xyz="${x} ${y} .36" rpy="0 0.0 0.0"/>
-        <parent link="base_link"/>
-        <child link="Wcrossbeam_${name}_link"/>
-        <axis xyz="0.0 0.0 0.0"/>
-    </joint>
-</xacro:macro>
-<xacro:Wcrossbeam name="left1"  x="0.0" y =" 0.70"/>
-<xacro:Wcrossbeam name="left2"  x="0.0" y =" 0.824"/>
-<xacro:Wcrossbeam name="right1"  x="0.0" y =" -0.70"/>
-<xacro:Wcrossbeam name="right2"  x="0.0" y =" -0.824"/>
 <!-- All Wheel links and joints -->
-<xacro:macro name="wheel" params="name x y">
+<xacro:macro name="wheel" params="name x y yaw">
     <link name="wheel_${name}_link">
         <inertial>
-            <origin xyz="0.0 0.0 0.0" rpy="0.0 0.0 0.0"/>
-            <mass value="0.5"/>
-            <inertia ixx="0.0" ixy="0.0" ixz="0.0" iyy="0.0" iyz="0.0" izz="0.0"/>
-        </inertial>
-        <visual name="">
-            <origin xyz="0.0 0.0 0.0" rpy="0.0 0.0 0.0"/>
-            <geometry>
-                <mesh filename="package://amiga_cmu_description/meshes/hub/hub.obj" scale="1.0 1.0 1.0"/>
-            </geometry>
-            <material name="black">
-                <color rgba=".0 .0 0.0 1.0"/>
-            </material>
-        </visual>
-        <collision>
-            <origin xyz="0.0 0.0 0.0" rpy="0.0 0.0 0.0"/>
-            <geometry>
-                <mesh filename="package://amiga_cmu_description/meshes/hub/hub.obj" scale="1.0 1.0 1.0"/>
+            <origin xyz="0.0 0.0 0.0" rpy="0.0 0.0 ${yaw}"/>
+            <mass value="0.5"/>
+            <inertia ixx="0.0" ixy="0.0" ixz="0.0" iyy="0.0" iyz="0.0" izz="0.0"/>
+        </inertial>
+        <visual name="">
+            <origin xyz="0.0 0.0 0.0" rpy="0.0 0.0 ${yaw}"/>
+            <geometry>
+                <mesh filename="package://amiga_cmu_description/meshes/test_hub/test_hub.obj" scale="1.0 1.0 1.0"/>
+            </geometry>
+            <material name="black">
+                <color rgba=".0 .0 0.0 1.0"/>
+            </material>
+        </visual>
+        <collision>
+            <origin xyz="0.0 0.0 0.0" rpy="0.0 0.0 ${yaw}"/>
+            <geometry>
+                <mesh filename="package://amiga_cmu_description/meshes/test_hub/test_hub.obj" scale="1.0 1.0 1.0"/>
             </geometry>
         </collision>
@@ -136,9 +67,80 @@
 </xacro:macro>
 <!-- Wheel Creating using macros -->
-<xacro:wheel name="rear_right"  x="0.6096" y =" 0.762"/>
-<xacro:wheel name="front_right" x="-0.6096" y =" 0.762"/>
-<xacro:wheel name="front_left"  x="-0.6096" y =" -0.762"/>
-<xacro:wheel name="rear_left"   x="0.6096" y =" -0.762"/>
-<xacro:macro name="tire" params="name x y">
+<xacro:wheel name="rear_right"  x="0.6096" y =" 0.762" yaw = "3.141"/>
+<xacro:wheel name="front_right" x="-0.6096" y =" 0.762" yaw = "3.141"/>
+<xacro:wheel name="front_left"  x="-0.6096" y =" -0.762" yaw = "0.0"/>
+<xacro:wheel name="rear_left"   x="0.6096" y =" -0.762" yaw = "0.0"/>
+<xacro:macro name="clamp" params="name">
+	<link name="clamp_${name}_link">
+        <inertial>
+            <origin xyz="0.0 0.0 0.0" rpy="0.0 0.0 0.0"/>
+            <mass value="0.5"/>
+            <inertia ixx="0.0" ixy="0.0" ixz="0.0" iyy="0.0" iyz="0.0" izz="0.0"/>
+        </inertial>
+        <visual name="">
+            <origin xyz="0.0 0.0 0.0" rpy="0.0 0.0 0.0"/>
+            <geometry>
+                <mesh filename="package://amiga_cmu_description/meshes/clamp/clamp.obj" scale="1.0 1.0 1.0"/>
+            </geometry>
+            <material name="black">
+                <color rgba=".0 .0 0.0 1.0"/>
+            </material>
+        </visual>
+        <collision>
+            <origin xyz="0.0 0.0 0.0" rpy="0.0 0.0 0.0"/>
+            <geometry>
+                <mesh filename="package://amiga_cmu_description/meshes/clamp/clamp.obj" scale="1.0 1.0 1.0"/>
+            </geometry>
+        </collision>
+    </link>
+    <joint name="clamp_${name}_joint" type="fixed">
+        <origin xyz="0.0 0.0 .395" rpy="0 0.0 0.0"/>
+        <parent link="wheel_${name}_link"/>
+        <child link="clamp_${name}_link"/>
+        <axis xyz="0.0 0.0 0.0"/>
+    </joint>
+</xacro:macro>
+<xacro:clamp name="rear_right" />
+<xacro:clamp name="front_right"/>
+<xacro:clamp name="front_left" />
+<xacro:clamp name="rear_left"  />
+<!-- All crossbeams links and joints -->
+<xacro:macro name="crossbeam" params="name x y z yaw ">
+    <link name="crossbeam_${name}_link">
+        <inertial>
+            <origin xyz="0.0 0.0 0.0" rpy="0.0 0.0 ${yaw}"/>
+            <mass value="0.5"/>
+            <inertia ixx="0.0" ixy="0.0" ixz="0.0" iyy="0.0" iyz="0.0" izz="0.0"/>
+        </inertial>
+        <visual name="">
+            <origin xyz="0.0 0.0 0.0" rpy="0.0 0.0 ${yaw}"/>
+            <geometry>
+                <mesh filename="package://amiga_cmu_description/meshes/LCrossbeam/LCrossbeam.obj" scale="1.0 1.3 1.0"/>
+            </geometry>
+            <material name="black">
+                <color rgba=".0 .0 0.0 1.0"/>
+            </material>
+        </visual>
+        <collision>
+            <origin xyz="0.0 0.0 0.0" rpy="0.0 0.0 ${yaw}"/>
+            <geometry>
+                <mesh filename="package://amiga_cmu_description/meshes/LCrossbeam/LCrossbeam.obj" scale="1.0 1.3 1.0"/>
+            </geometry>
+        </collision>
+    </link>
+    <joint name="crossbeam_${name}_joint" type="fixed">
+        <origin xyz="${x} ${y} ${z}" rpy="0 0.0 0.0"/>
+        <parent link="base_link"/>
+        <child link="crossbeam_${name}_link"/>
+        <axis xyz="0.0 0.0 0.0"/>
+    </joint>
+</xacro:macro>
+<xacro:crossbeam name="back"  x="0.6096" y =" 0.0" z = "0.417" yaw = "0.0" />
+<xacro:crossbeam name="front"  x="-0.6096" y =" 0.0" z = "0.417" yaw = "0.0" />
+<xacro:crossbeam name="left1"  x="0.0" y =" 0.70" z = "0.36" yaw = "1.571" />
+<xacro:crossbeam name="left2"  x="0.0" y =" 0.824" z = "0.36" yaw = "1.571" />
+<xacro:crossbeam name="right1"  x="0.0" y =" -0.70" z = "0.36" yaw = "1.571" />
+<xacro:crossbeam name="right2"  x="0.0" y =" -0.824" z = "0.36" yaw = "1.571" />
+<xacro:macro name="tire" params="name">
 	<link name="tire_${name}_link">
         <inertial>
@@ -164,14 +166,14 @@
     </link>
     <joint name="tire_${name}_joint" type="continuous">
-        <origin xyz="${x} ${y} .0" rpy="0 0.0 0.0"/>
-        <parent link="base_link"/>
+        <origin xyz="0.0 0.0 0.0" rpy="0 0.0 0.0"/>
+        <parent link="wheel_${name}_link"/>
         <child link="tire_${name}_link"/>
         <axis xyz="0.0 1.0 0.0"/>
     </joint>
 </xacro:macro>
-<xacro:tire name="rear_right"  x="0.6096" y =" 0.762"/>
-<xacro:tire name="front_right" x="-0.6096" y =" 0.762"/>
-<xacro:tire name="front_left"  x="-0.6096" y =" -0.762"/>
-<xacro:tire name="rear_left"   x="0.6096" y =" -0.762"/>
+<xacro:tire name="rear_right"  />
+<xacro:tire name="front_right" />
+<xacro:tire name="front_left"  />
+<xacro:tire name="rear_left"   />
 <xacro:arg name="prefix" default=""/>
   <xacro:arg name="ros_namespace" default="xarm"/>
@@ -194,5 +196,5 @@
   <xacro:arg name="geometry_mesh_tcp_xyz" default="0 0 0"/>
   <xacro:arg name="geometry_mesh_tcp_rpy" default="0 0 0"/>
-  <xacro:arg name="add_ee" default="true"/>
+  <xacro:arg name="add_ee" default="false"/>
   <xacro:arg name="model1300" default="false"/>
   <!-- load xarm6 robot -->
